Commit message: Started on Gazebo integration. STATUS: robot not moving in sim. pausible cause conflict in joint_state publishers

File: src/kuka_experimental/kuka_kr16_gazebo/urdf/kuka_kr16_2.xacro (robot description, xacro)
@@ -1,4 +1,4 @@
 <?xml version="1.0" ?>
-<robot name="kuka_kr16" xmlns:xacro="http://ros.org/wiki/xacro">
+<robot name="kuka_kr16_2" xmlns:xacro="http://ros.org/wiki/xacro">
   <xacro:include filename="$(find kuka_kr16_gazebo)/urdf/kuka_kr16_2_macro.xacro"/>
   <xacro:kuka_kr16_gazebo prefix=""/>

File: src/kuka_experimental/kuka_kr16_support/urdf/kr16_2_macro.xacro (robot description, xacro)
@@ -5,4 +5,9 @@
     <!-- base link -->
     <link name="${prefix}base_link">
+      <inertial>
+        <origin xyz="0 0 0" rpy="0 0 0"/>
+        <mass value="2"/>
+        <inertia ixx="0" ixy="0" ixz="0" iyy="0" iyz="0" izz="0" />
+      </inertial>
       <visual>
         <origin xyz="0 0 0" rpy="0 0 0"/>
@@ -149,5 +154,5 @@
       <child link="${prefix}link_1"/>
       <axis xyz="0 0 -1"/>
-      <limit effort="0" lower="${radians(-185)}" upper="${radians(185)}" velocity="${radians(156)}"/>
+      <limit effort="1" lower="${radians(-185)}" upper="${radians(185)}" velocity="${radians(156)}"/>
     </joint>
     <!-- joint 2 (A2) -->
@@ -157,5 +162,5 @@
       <child link="${prefix}link_2"/>
       <axis xyz="0 1 0"/>
-      <limit effort="0" lower="${radians(-155)}" upper="${radians(35)}" velocity="${radians(156)}"/>
+      <limit effort="1" lower="${radians(-155)}" upper="${radians(35)}" velocity="${radians(156)}"/>
     </joint>
     <!-- joint 3 (A3) -->
@@ -165,5 +170,5 @@
       <child link="${prefix}link_3"/>
       <axis xyz="0 1 0"/>
-      <limit effort="0" lower="${radians(-130)}" upper="${radians(154)}" velocity="${radians(156)}"/>
+      <limit effort="1" lower="${radians(-130)}" upper="${radians(154)}" velocity="${radians(156)}"/>
     </joint>
     <!-- joint 4 (A4) -->
@@ -173,5 +178,5 @@
       <child link="${prefix}link_4"/>
       <axis xyz="-1 0 0"/>
-      <limit effort="0" lower="${radians(-350)}" upper="${radians(350)}" velocity="${radians(330)}"/>
+      <limit effort="1" lower="${radians(-350)}" upper="${radians(350)}" velocity="${radians(330)}"/>
     </joint>
     <!-- joint 5 (A5) -->
@@ -181,5 +186,5 @@
       <child link="${prefix}link_5"/>
       <axis xyz="0 1 0"/>
-      <limit effort="0" lower="${radians(-130)}" upper="${radians(130)}" velocity="${radians(330)}"/>
+      <limit effort="1" lower="${radians(-130)}" upper="${radians(130)}" velocity="${radians(330)}"/>
     </joint>
     <!-- joint 6 (A6) -->
@@ -189,5 +194,5 @@
       <child link="${prefix}link_6"/>
       <axis xyz="-1 0 0"/>
-      <limit effort="0" lower="${radians(-350)}" upper="${radians(350)}" velocity="${radians(615)}"/>
+      <limit effort="1" lower="${radians(-350)}" upper="${radians(350)}" velocity="${radians(615)}"/>
     </joint>
     <!-- tool frame - fixed frame -->
